File: Electronics/PIMD604/PIMD604-Sheet2.kicad_sch (KiCad schematic)
At the start: 39 parts, among them J11 Conn_01x08_Pin, J12 Screw_Terminal_01x02, SW5 SW_MEC_5G, SW6 SW_MEC_5G, U11 TL074, U12 74LS04, U18 LT6203

Commit message: starting /clean
Other:
- note added: "16/06/2026 copied unused symobols and nets to this page, HOWEVER it reannotated all the references. Needs correction from v6.01 schem"
Changed lines of the file:
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@@
+		)
+	)
+	(text "16/06/2026\ncopied unused symobols and nets to this page, \nHOWEVER it reannotated all the references.  \nNeeds correction from v6.01 schem"
+		(exclude_from_sim no)
+		(at 189.484 38.354 0)
+		(effects
+			(font
+				(size 2.032 2.032)
+			)
+			(justify left bottom)
 		)
 	)
