File: Electronics/PIMD604/PIMD604.kicad_sch (KiCad schematic)
At the start: 86 parts, among them J1 Screw_Terminal_01x02, J2 Screw_Terminal_01x02, J3 Screw_Terminal_01x02, J4 RFShield_OnePiece, Q1 IRF610, SW3 SW_SPDT, U1 LM7815, U10 RP2040-Zero, U2 L7812, U3 LT6203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

Commit message: starting /clean
Parts:
- removed D1: 1N5817, _MM-footprints:D_DO-41_SOD81_P10.16mm_Horizontal, symbol Diode:1N5817
- removed R26: 0R, _MM-footprints:Resistor, symbol Device:R_US
- C18: value 2200u -> 4700u
- C19: Field4 16V -> 25V
- D2: value 1N4733 -> 1N4732; Field4 5V1 -> 4V7
- D3: value 1N5817 -> 1N5819
- R1: value 1k8 -> 1k3
- R10: value 270R -> 0R
- R12, R13: value 4R7 -> 0R
- R23: value 2k7 -> 18k
- R9: value 10k -> 4k7
- U1: value LM7815 -> L7815CV
- U2: value L7812 -> L7812CV
- U9: value LM7805 -> L7805CV
Connections:
- net COMMS-TX is gone; now on net ADCSEL0: TP9.1, U10.13 (GP12)
- net TX-COIL-NEG: now also J1.2 (Pin_2); no longer J1.1 (Pin_1)
- net TX-COIL-POS: now also J1.1 (Pin_1); no longer J1.2 (Pin_2)
- net ADCSEL0: now reaches U6.11 (SEL0)
- net at COIL1. (SB): now also J4.
- net at U7.6 (NC): now also C14.1
Other:
- note added: "5V PRECISION REFERENCE FOR ADC"
- note added: "Q1 Note Drain and Gate reversed on PCB, correct in newer version"
- note added: "R12/R13 originally 4.7R 5W resistors to speed up sample time, according to expert sources, however in my testing but works better without."
- note added: "[-0.48V to +5.11V]"
- note added: "[-0.55V to +5.32V]"
- note added: "[0.44V to 11.47V fall time 733ns]"
- note added: "[1.6V to 3.2V]"
- note added: "[1.6V]"
- note added: "[40 uS pulse: -15V to +135V]"
- note added: "[40 uS pulse: -18V to +265V]"
- note added: "[Red annotations in [] brackets dentore field measurements]"
- note added: "[at 10kHz 40 uS pulses, 500mA from bench supply at 20V]"
- note added: "magnet wire, enamel insul. ID 400mm eliptical 0.5mm x 14T = 1.8R (24 AWG) step resp. 544kHz,"
- note added: "wirewrap wire, teflon insul. ID 400mm round 0.25mm x 50T = 19.9R (30 AWG) step resp. 164kHz,"
- note removed: "5V PRECISION REFERENCE"
- note removed: "IRF610 LIMIT <10A <300us <2%"
- note removed: "[-0.7 to +5.1]"
- note removed: "[0 to +5.1]"
- note removed: "[1.6 > 10.7]"
- note removed: "[1.7 to 3.4]"
- note removed: "magnet wire, enamel insul. ID 400mm eliptical 0.5mm x 14T = 1.8R (24 AWG) step resp. 544kHz, calcs: 275uH, 266pF, Rd = 469 (but 220R better ?)"
- note removed: "wirewrap wire, teflon insul. ID 400mm round 0.25mm x 50T = 19.9R (30 AWG) step resp. 164kHz, calc: 3.5mH, 311pF, Rd = 1822"
- moved on the sheet: C10, C16, C19, C4, R14, R17, R18, R20, R21, R22, R23, R27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

Commit message: now maintaining CHANGELOG
Connections:
- net at COIL1. (SB): now also J4.
- net at U7.6 (NC): now also C14.1
Other:
- note added: "A / DRL : 32 bits filtered B / BUSY : 22 bits raw The 22-bit composite code consists of a 14-bit code representing the differential voltage and an 8-bit code representing the common mode voltage."
- note removed: "A / DRL : 32 bits filtered B / BUSY : 22 bits raw"
Changed lines of the file:
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@@
 		)
 	)
-	(text "A / DRL  : 32 bits filtered\nB / BUSY : 22 bits raw"
+	(text "A / DRL  : 32 bits filtered\nB / BUSY : 22 bits raw \n\nThe 22-bit composite code consists of a\n14-bit code representing the differential voltage and an\n8-bit code representing the common mode voltage."
 		(exclude_from_sim no)
-		(at 219.71 175.26 0)
+		(at 226.06 185.166 0)
 		(effects
 			(font
